File: thelio-io.kicad_sch (KiCad schematic)
At the start: 28 parts, among them J1 CDR-04-GS, Y1 ECS-160-18-23G-JGN-TR

Commit message: v2 with RP2040
Parts:
- removed AVR1: AT90USB646-MUR, Package_DFN_QFN:QFN-64-1EP_9x9mm_P0.5mm_EP7.5x7.5mm, symbol MCU_Microchip_AVR:AT90USB646-M
- removed C2, C3: 22 pF, Capacitor_SMD:C_0402_1005Metric, symbol Device:C
- removed C8: 1 uF, Capacitor_SMD:C_0402_1005Metric, symbol Device:C
- removed ICSP1: 54202-S0803LF, Connector_PinHeader_2.54mm:PinHeader_2x03_P2.54mm_Vertical_SMD, symbol Connector_Generic:Conn_02x03_Odd_Even
- removed MUX1, MUX2, MUX3, MUX4: SN74LVC2G157DCUR, Package_SO:VSSOP-8_2.4x2.1mm_P0.5mm, symbol 74xGxx:74LVC2G157
- removed Y1: ECS-160-18-23G-JGN-TR, Crystal:Crystal_SMD_0603-2Pin_6.0x3.5mm, symbol Device:Crystal
- added C10, C11: 1 uF, kicad_pcb:C_0402_1005Metric, symbol Device:C
- added C7, C9: 27 pF, kicad_pcb:C_0402_1005Metric, symbol Device:C
- added J6: SWD_TH, Connector_PinHeader_2.54mm:PinHeader_1x04_P2.54mm_Vertical, symbol Connector_Generic:Conn_01x04
- added Q1, Q10, Q11, Q12, Q13, Q2, Q3, Q4, Q5, Q6, Q7, Q8, Q9: BSS138PW, Package_TO_SOT_SMD:SOT-323_SC-70, symbol Transistor_FET:2N7002
- added R10, R11, R12, R13, R14, R15, R16, R17, R22, R23, R4, R5, R9: 5.1 k, kicad_pcb:R_0402_1005Metric, symbol Device:R
- added R18, R19, R20, R21: DNP, kicad_pcb:R_0402_1005Metric, symbol Device:R
- added R6: 1 k, kicad_pcb:R_0402_1005Metric, symbol Device:R
- added R7, R8: 27, kicad_pcb:R_0402_1005Metric, symbol Device:R
- added SW1, SW2: SKRPACE010, kicad_pcb:SW_SPST_PTS810, symbol Switch:SW_Push
- added U1: W25Q16JVSSIQ, Package_SO:SOIC-8_5.23x5.23mm_P1.27mm, symbol QSPI_flash:W25Q16JVSSIQ
- added U2: RP2040, kicad_pcb:QFN-56-RP2040, symbol RP2040:RP2040
- added U3: LP5907MFX-3.3, Package_TO_SOT_SMD:SOT-23-5, symbol Regulator_Linear:LP5907MFX-3.3
- added Y2: RH100-12.000-18-2030-TR, Oscillator:Oscillator_SMD_SeikoEpson_SG8002CE-4Pin_3.2x2.5mm, symbol Device:Crystal_GND24
- C1: footprint Capacitor_SMD:C_0402_1005Metric -> kicad_pcb:C_0402_1005Metric; Manufacturer generic -> (none)
- PWBT1: value TL3342F260QG -> SKRPACE010; footprint Button_Switch_SMD:SW_SPST_TL3342 -> kicad_pcb:SW_SPST_PTS810; Manufacturer E-Switch (generic equivalent OK) -> Alps (generic equivalent OK)
- R1, R2: value 22 -> 5.1 k; footprint Resistor_SMD:R_0603_1608Metric -> kicad_pcb:R_0402_1005Metric
Connections:
- net OC1A is gone; now on net VCC: R3.1
- net UCAP is gone; now on net GND: C1.1
- net ADC0: now also R9.2, U2.38 (GPIO26_ADC0); no longer PFP1.1, PMB1.1, PWBT1.1 (A)
- net ADC1: now also R10.1, U2.39 (GPIO27_ADC1); no longer PFP1.2, PMB1.2, PWBT1.2 (B)
- net ADC2: now also R2.2, U2.40 (GPIO28_ADC2); no longer PMB1.3 (K)
- net ADC3: now also R11.1, U2.41 (GPIO29_ADC3); no longer PMB1.4 (A)
- net D+: now also R7.1; no longer R1.1
- net D-: now also R8.1; no longer R2.1
- net DR+: now also R7.2, U2.47 (USB_DP); no longer R1.2
- net DR-: now also R8.2, U2.46 (USB_DM); no longer R2.2
- net GND: now also C10.1, C11.1, C7.2, C9.2, J6.4 (Pin_4), Q1.2 (S), Q10.2 (S), Q11.2 (S), Q12.2 (S), Q13.2 (S), Q2.2 (S), Q3.2 (S), Q4.2 (S), Q5.2 (S), Q6.2 (S), Q7.2 (S), Q8.2 (S), Q9.2 (S), R13.2, R14.2, R15.2, R16.2, R17.2, SW1.1, SW2.1, U1.4 (GND), U2.19 (TESTEN), U2.57 (GND), U3.2 (GND), Y2.2, Y2.4; no longer C1.2, PFP1.3 (K)
- net PWMIN: now also R1.2, Q6.1 (G)
- net VCC: now also R18.1, R19.1, R20.1, R21.1, U3.1 (IN), U3.3 (EN); no longer C4.1, C5.1
- net at FANOUT2.4 (PWM): now also Q4.3 (D), Q9.3 (D), R19.2
- net at FANOUT3.4 (PWM): now also Q10.3 (D), Q3.3 (D), R20.2
- net at FANOUT1.4 (PWM): now also Q5.3 (D), Q8.3 (D), R18.2
- net at FANOUT4.4 (PWM): now also Q11.3 (D), Q2.3 (D), R21.2
- net ADC4 renamed TACH0
- net TACH0: now also Q13.1 (G), R23.2, U2.7 (GPIO5); no longer FANIN1.3 (Tacho)
- net ADC5 renamed TACH1
- net TACH1: now also U2.9 (GPIO7)
- net ADC6 renamed TACH2
- net TACH2: now also U2.12 (GPIO9)
- net ADC7 renamed TACH3
- net TACH3: now also U2.14 (GPIO11)
- new net: PMB1.3 (K), R2.1
- new net: PMB1.4 (A), R11.2
- new net +3V3: C11.2, C4.1, C5.1, J6.1 (Pin_1), R1.1, R12.1, R22.1, R23.1, R4.1, R5.1, U1.8 (VCC), U2.1 (IOVDD), U2.10 (IOVDD), U2.22 (IOVDD), U2.33 (IOVDD), U2.42 (IOVDD), U2.43 (ADC_AVDD), U2.44 (VREG_IN), U2.48 (USB_VDD), U2.49 (IOVDD), U3.5 (OUT)
- new net DIS_PWMIN: Q7.1 (G), R13.1, U2.15 (GPIO12)
- new net PB1: PFP1.2, PMB1.2, PWBT1.2 (B), R10.2
- new net PB2: PFP1.1, PMB1.1, PWBT1.1 (A), R9.1
- new net PLED: Q1.1 (G), U2.16 (GPIO13)
- new net PWM0: Q5.1 (G), R14.1, U2.27 (GPIO16)
- new net PWM1: Q4.1 (G), R15.1, U2.28 (GPIO17)
- new net PWM2: Q3.1 (G), R16.1, U2.29 (GPIO18)
- new net PWM3: Q2.1 (G), R17.1, U2.30 (GPIO19)
- new net QD0: U1.5 (IO0/DI), U2.53 (QSPI_SD0)
- new net QD1: U1.2 (IO1/DO), U2.55 (QSPI_SD1)
- new net QD2: U1.3 (IO2/~{WP}), U2.54 (QSPI_SD2)
- new net QD3: U1.7 (IO3/~{HOLD}), U2.51 (QSPI_SD3)
- new net QSCK: U1.6 (CLK), U2.52 (QSPI_SCLK)
- new net RUN: R4.2, SW1.2, U2.26 (RUN)
- new net SWCLK: J6.3 (Pin_3), U2.24 (SWCLK)
- new net SWDIO: J6.2 (Pin_2), U2.25 (SWD)
- new net TACH0_MB: FANIN1.3 (Tacho), Q12.3 (D)
- new net VCORE: C1.2, C10.2, U2.23 (DVDD), U2.45 (VREG_VOUT), U2.50 (DVDD)
- new net XIN: C7.1, U2.20 (XIN), Y2.3
- new net XOUT: C9.1, R6.2, Y2.1
- new net XOUT1: R6.1, U2.21 (XOUT)
- new net ~{PLED}: PFP1.3 (K), Q1.3 (D)
- new net ~{PWMIN}: Q10.1 (G), Q11.1 (G), Q6.3 (D), Q7.3 (D), Q8.1 (G), Q9.1 (G), R12.2
- new net ~{QCS}: R5.2, SW2.2, U1.1 (CS#), U2.56 (QSPI_SS)
- new net ~{TACH0}: Q12.1 (G), Q13.3 (D), R22.2
- no-connect marks 37 -> 3
Other:
- note added: "Alt: Yangxing X322512MSB4SI"
- note added: "Alternate 4 wire PWM fan documentation: https://www.noctua.at/pub/media/wysiwyg/Noctua_PWM_specifications_white_paper.pdf"
- note added: "DFU: hold while releasing reset for USB DFU"
- note added: "Lighted power button on front panel The LED in the button has an integrated resistor, is specified for 6 V. 5V is OK with reduced brighness R3 can be adjusted to vary brightness of the power LED."
- note added: "PMB1 connects to the motherboard power button/LED connector The 4 ADCs are used to sense the LED and power button state series resistors provide protection against 5 V"
- note added: "PWM0A PWM0B"
- note added: "PWM1A PWM1B"
- note added: "PWM2B"
- note added: "PWM3B"
- note added: "PWM4B"
- note added: "PWM5B"
- note added: "PWM6B"
- note added: "Reset"
- note added: "Serial Wire Debug"
- note added: "These pullup resistors are optional. They are not allowed according to the Intel PWM fan spec, the Noctua PWM fan spec suggests they should be used."
- note added: "This connects to a motherboard fan header, is not a fan"
- note added: "button on PCB"
- note added: "place 2 series termination resistors close to RP2040"
- note added: "to use the motherboard PWM, set PWM0-3 low, DIS_PWMIN low to use the microcontroller PWM, drive PWM on PWM0-3, set DIS_PWMIN high, PWM0-3 are inverted. Constant logic 1 is minimum fan speed, constant logic 0 is maximum fan speed."
- note removed: "OC1B"
- note removed: "SS"
- moved on the sheet: C4, C5, C6, F1, FANIN1, FANOUT1, FANOUT2, FANOUT3, FANOUT4, J1, PFP1, PMB1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
