File: thelio-io-sata.kicad_sch (KiCad schematic)
At the start: 5 parts

Commit message: thelio-io-sata 2.0 add SMT standoffs, move connector locations
Parts:
- added H1, H2, H3, H4, H5, H6: SMTSOM330STR, SMTSO:SMTSO-M3-3, symbol Mechanical:MountingHole_Pad
Connections:
- net GND: now also H1.1, H2.1, H3.1, H4.1, H5.1, H6.1
